File: CustomBMS.kicad_sch (KiCad schematic)
At the start: 0 parts

Commit message: second changes in bms monitoring
Other:
- sheet MCU+Monitor IC renamed Monitor IC CONFIG
- added sheet Charger and Load detection (charger&load_detection.kicad_sch)
- added sheet MCU Config (MCU_config.kicad_sch)
- sheet Monitor IC CONFIG ports: added ALERT_B, Alert_B_U, CHG_B, CHG_U, DSG_B, DSG_U, I2C_CTRL_B, I2C_CTRL_B_U, I2C_CTRL_U, SCL_MCU, SDA_MCU; removed none

Commit message: home changes
Other:
- added sheet Power Supply (power.kicad_sch)
- sheet MCU Config ports: added 3.3, GND, I2C_SCL, I2C_SDA; removed none
- sheet Monitor IC CONFIG ports: added CHG_ACTIVATE, GND_B, GND_U, VCC_B; removed none
Changed lines of the file:
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@@
+	)
+	(sheet
+		(at 228.6 24.13)
+		(size 41.91 39.37)
+		(fields_autoplaced yes)
+		(stroke
+			(width 0.1524)
+			(type solid)
+		)
+		(fill
+			(color 0 0 0 0.0000)
+		)
+		(property "Sheetname" "Power Supply"
+			(at 228.6 23.4184 0)
+			(effects
+				(font
+					(size 1.27 1.27)
+				)
+				(justify left bottom)
+			)
+		)
+		(property "Sheetfile" "power.kicad_sch"
+			(at 228.6 64.0846 0)
+			(effects
+				(font
+					(size 1.27 1.27)
+				)
+				(justify left top)
+			)
+		)
+		(pin "GND" input
+			(at 270.51 35.56 0)
+			(effects
+				(font
+					(size 1.27 1.27)
+				)
+				(justify right)
+			)
+		)
+		(pin "3.3V" input
+			(at 270.51 45.72 0)
+			(effects
+				(font
+					(size 1.27 1.27)
+				)
+				(justify right)
+			)
+		)
+		(pin "12V" input
+			(at 228.6 39.37 180)
+			(effects
+				(font
+					(size 1.27 1.27)
+				)
+				(justify left)
+			)
+		)
+		(instances
+			(project "CustomBMS"
+				(path "/422fc8bd-c42e-475a-86fa-949c078f7358"
+					(page "6")
+				)
+			)
+		)
 	)
 	(sheet
@@
 			)
 		)
+		(pin "GND" input
+			(at 173.99 62.23 180)
+			(effects
+				(font
+					(size 1.27 1.27)
+				)
+				(justify left)
+			)
+		)
+		(pin "3.3" input
+			(at 173.99 69.85 180)
+			(effects
+				(font
+					(size 1.27 1.27)
+				)
+				(justify left)
+			)
+		)
+		(pin "I2C_SCL" input
+			(at 173.99 76.2 180)
+			(effects
+				(font
+					(size 1.27 1.27)
+				)
+				(justify left)
+			)
+		)
+		(pin "I2C_SDA" input
+			(at 173.99 82.55 180)
+			(effects
+				(font
+					(size 1.27 1.27)
+				)
+				(justify left)
+			)
+		)
 		(instances
 			(project "CustomBMS"
@@
 			)
 		)
+		(pin "CHG_ACTIVATE" input
+			(at 44.45 106.68 180)
+			(effects
+				(font
+					(size 1.27 1.27)
+				)
+				(justify left)
+			)
+		)
+		(pin "GND_B" input
+			(at 44.45 115.57 180)
+			(effects
+				(font
+					(size 1.27 1.27)
+				)
+				(justify left)
+			)
+		)
+		(pin "GND_U" input
+			(at 44.45 124.46 180)
+			(effects
+				(font
+					(size 1.27 1.27)
+				)
+				(justify left)
+			)
+		)
+		(pin "VCC_B" input
+			(at 44.45 137.16 180)
+			(effects
+				(font
+					(size 1.27 1.27)
+				)
+				(justify left)
+			)
+		)

Commit message: schematic v0
Parts:
- added J4: Conn_01x10_Pin, symbol Connector:Conn_01x10_Pin
- added J5: Conn_01x12_Pin, symbol Connector:Conn_01x12_Pin
Connections:
- new net Monitor IC CONFIG/BATT_1+: J5.2 (Pin_2)
- new net Monitor IC CONFIG/BATT_10+: J5.11 (Pin_11)
- new net Monitor IC CONFIG/BATT_11+: J5.12 (Pin_12)
- new net Monitor IC CONFIG/BATT_12+: J4.1 (Pin_1)
- new net Monitor IC CONFIG/BATT_13+: J4.2 (Pin_2)
- new net Monitor IC CONFIG/BATT_14+: J4.3 (Pin_3)
- new net Monitor IC CONFIG/BATT_15+: J4.4 (Pin_4)
- new net Monitor IC CONFIG/BATT_16+: J4.5 (Pin_5)
- new net Monitor IC CONFIG/BATT_17+: J4.6 (Pin_6)
- new net Monitor IC CONFIG/BATT_18+: J4.7 (Pin_7)
- new net Monitor IC CONFIG/BATT_19+: J4.8 (Pin_8)
- new net Monitor IC CONFIG/BATT_1_NEG: J5.1 (Pin_1)
- new net Monitor IC CONFIG/BATT_2+: J5.3 (Pin_3)
- new net Monitor IC CONFIG/BATT_20+: J4.9 (Pin_9)
- new net Monitor IC CONFIG/BATT_21+: J4.10 (Pin_10)
- new net Monitor IC CONFIG/BATT_3+: J5.4 (Pin_4)
- new net Monitor IC CONFIG/BATT_4+: J5.5 (Pin_5)
- new net Monitor IC CONFIG/BATT_5+: J5.6 (Pin_6)
- new net Monitor IC CONFIG/BATT_6+: J5.7 (Pin_7)
- new net Monitor IC CONFIG/BATT_7+: J5.8 (Pin_8)
- new net Monitor IC CONFIG/BATT_8+: J5.9 (Pin_9)
- new net Monitor IC CONFIG/BATT_9+: J5.10 (Pin_10)
Other:
- sheet Charge and discharge mosfets ports: added CHG_B, CHG_U, DSG_B, DSG_U, GND_B, GND_U, Logic_ref, Turn_ON _gate_V; removed BAT+, CHG, DSG, PORT+
- sheet MCU Config ports: added ALERT_B, ALERT_B_U, CHG_DET, I2C_CTRL_B, I2C_CTRL_B_U, I2C_CTRL_U, LOAD_RM_DETECT, PDSG; removed none
- sheet Monitor IC CONFIG ports: added BATT_1+, BATT_10+, BATT_11+, BATT_12+, BATT_13+, BATT_14+, BATT_15+, BATT_16+, BATT_17+, BATT_18+, BATT_19+, BATT_1_NEG, BATT_2+, BATT_20+, BATT_21+, BATT_3+, BATT_4+, BATT_5+, BATT_6+, BATT_7+, BATT_8+, BATT_9+, SHUNT_N, SHUNT_P, TS1_B, VC5X_B; removed none

Commit message: Demo commit
Parts:
- added J6: Conn_01x02_Socket, symbol Connector:Conn_01x02_Socket
- added J7: Conn_01x01_Socket, symbol Connector:Conn_01x01_Socket
- added J8: Conn_01x01, symbol Connector_Generic:Conn_01x01
Connections:
- net Charge and discharge mosfets/CHG+: now also J8.1 (Pin_1)
- net Power Supply/12V: now also J6.1 (Pin_1)
- net Monitor IC CONFIG/BATT_1_NEG renamed BATT-
- net Monitor IC CONFIG/BATT_21+ renamed BATT+
- new net GND_B: J6.2 (Pin_2)
- new net PACK-: J7.1 (Pin_1)
