File: MCU_config.kicad_sch (KiCad schematic)
At the start: 1 part, among them IC1 STM32F401RET6

Commit message: home changes
Parts:
- removed IC1: STM32F401RET6, QFP50P1200X1200X160-64N, symbol STM32f401REt6:STM32F401RET6
- added C25: 10uF, Capacitor_SMD:C_1206_3216Metric, symbol Device:C
- added C26, C27, C28, C29, C34: 100nF, Capacitor_SMD:C_0402_1005Metric, symbol Device:C
- added C30, C31, C32, C33: 22pF, Capacitor_SMD:C_0402_1005Metric, symbol Device:C
- added D38: LED, LED_THT:LED_D2.0mm_W4.0mm_H2.8mm_FlatTop, symbol Device:LED
- added J1: Conn_02x03_Odd_Even, Connector_PinHeader_2.54mm:PinHeader_2x03_P2.54mm_Vertical, symbol Connector_Generic:Conn_02x03_Odd_Even
- added J2: 8-1437565-1, 8-1437565:814375651, symbol 8-1437565:8-1437565-1
- added J3: Conn_01x02_Pin, Connector_PinHeader_2.54mm:PinHeader_1x02_P2.54mm_Vertical, symbol Connector:Conn_01x02_Pin
- added R88, R89: 100k, Resistor_SMD:R_0402_1005Metric, symbol Device:R
- added R90: 10k, Resistor_SMD:R_0402_1005Metric, symbol Device:R
- added R91: 330 ohm, Resistor_SMD:R_0201_0603Metric, symbol Device:R
- added U4: STM32F103C8Tx, Package_QFP:LQFP-48_7x7mm_P0.5mm, symbol MCU_ST_STM32F1:STM32F103C8Tx
- added U5: SN65HVD232, Package_SO:SOIC-8_3.9x4.9mm_P1.27mm, symbol Interface_CAN_LIN:SN65HVD232
- added Y1: Crystal_GND24_Small, Crystal:Crystal_SMD_3225-4Pin_3.2x2.5mm, symbol Device:Crystal_GND24_Small
- added Y2: Crystal_LSE_32.768kHz, Crystal:Crystal_SMD_3215-2Pin_3.2x1.5mm, symbol Device:Crystal
Connections:
- new net: J1.4 (Pin_4), R89.1
- new net: D38.2 (A), R91.1
- new net: R91.2, U4.2 (PC13)
- new net: J1.3 (Pin_3), R88.2
- new net 3.3: C25.1, C26.1, C27.1, C28.1, C29.1, J1.1 (Pin_1), J1.2 (Pin_2), R90.1, U4.24 (VDD), U4.36 (VDD), U4.48 (VDD), U4.9 (VDDA), U5.3 (VCC)
- new net BOOT0: R88.1, U4.44 (BOOT0)
- new net BOOT1: R89.2, U4.20 (PB2)
- new net CAN_Rx: U4.32 (PA11), U5.4 (R)
- new net CAN_Tx: U4.33 (PA12), U5.1 (D)
- new net GND: C25.2, C26.2, C27.2, C28.2, C29.2, C30.2, C31.2, C32.2, C33.2, C34.2, D38.1 (K), J1.5 (Pin_5), J1.6 (Pin_6), J2.3 (NO_1), J3.1 (Pin_1), U4.23 (VSS), U4.35 (VSS), U4.47 (VSS), U4.8 (VSSA), Y1.2, Y1.4
- new net I2C_SCL: U4.42 (PB6)
- new net I2C_SDA: U4.43 (PB7)
- new net RCC_OSC32_IN: C32.1, U4.3 (PC14), Y2.1
- new net RCC_OSC32_OUT: C33.1, U4.4 (PC15), Y2.2
- new net RCC_OSC_IN: C30.1, U4.5 (PD0), Y1.1
- new net RCC_OSC_OUT: C31.1, U4.6 (PD1), Y1.3
- new net RST: C34.1, J2.2 (COM_2), J3.2 (Pin_2), R90.2, U4.7 (NRST)

Commit message: schematic v0
Connections:
- net GND: now also U5.2 (GND)
- net PDSG: now reaches U4.11 (PA1)
- net ALERT_B: now reaches U4.18 (PB0)
- net ALERT_B_U: now reaches U4.19 (PB1)
- net CHG_DET: now reaches U4.25 (PB12)
- net LOAD_RM_DETECT: now reaches U4.29 (PA8)
- net I2C_CTRL_U: now reaches U4.39 (PB3)
- net I2C_CTRL_B: now reaches U4.40 (PB4)
- net I2C_CTRL_B_U: now reaches U4.41 (PB5)
Changed lines of the file:
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@@
+	(wire
+		(pts
+			(xy 158.75 97.79) (xy 172.72 97.79)
+		)
+		(stroke
+			(width 0)
+			(type default)
+		)
+	)
+	(wire
+		(pts
+			(xy 215.9 59.69) (xy 205.74 59.69)
+		)
+		(stroke
+			(width 0)
+			(type default)
+		)
+	)
 	(wire
 		(pts
@@
 	(wire
 		(pts
+			(xy 158.75 95.25) (xy 172.72 95.25)
+		)
+		(stroke
+			(width 0)
+			(type default)
+		)
+	)
+	(wire
+		(pts
 			(xy 193.04 49.53) (xy 190.5 49.53)
 		)
@@
 	(wire
 		(pts
+			(xy 161.29 87.63) (xy 172.72 87.63)
+		)
+		(stroke
+			(width 0)
+			(type default)
+		)
+	)
+	(wire
+		(pts
 			(xy 59.69 31.75) (xy 69.85 31.75)
 		)
@@
 	(wire
 		(pts
+			(xy 248.92 123.19) (xy 248.92 129.54)
+		)
+		(stroke
+			(width 0)
+			(type default)
+		)
+	)
+	(wire
+		(pts
 			(xy 40.64 77.47) (xy 40.64 62.23)
 		)
@@
 	(wire
 		(pts
+			(xy 162.56 85.09) (xy 172.72 85.09)
+		)
+		(stroke
+			(width 0)
+			(type default)
+		)
+	)
+	(wire
+		(pts
 			(xy 58.42 81.28) (xy 58.42 76.2)
 		)
@@
 	(wire
 		(pts
+			(xy 167.64 115.57) (xy 172.72 115.57)
+		)
+		(stroke
+			(width 0)
+			(type default)
+		)
+	)
+	(wire
+		(pts
 			(xy 49.53 142.24) (xy 54.61 142.24)
 		)
@@
 	(wire
 		(pts
+			(xy 205.74 77.47) (xy 209.55 77.47)
+		)
+		(stroke
+			(width 0)
+			(type default)
+		)
+	)
+	(wire
+		(pts
 			(xy 38.1 132.08) (xy 30.48 132.08)
 		)
@@
 		(pts
 			(xy 36.83 40.64) (xy 36.83 41.91)
+		)
+		(stroke
+			(width 0)
+			(type default)
+		)
+	)
+	(wire
+		(pts
+			(xy 158.75 92.71) (xy 172.72 92.71)
 		)
 		(stroke
@@
 	(label "BOOT1"
 		(at 67.31 134.62 180)
-		(fields_autoplaced yes)
 		(effects
 			(font
@@
 	(label "3.3DCV"
 		(at 91.44 31.75 180)
-		(fields_autoplaced yes)
 		(effects
 			(font
@@
 	(label "CAN_Tx"
 		(at 229.87 110.49 0)
-		(fields_autoplaced yes)
 		(effects
 			(font
@@
 	(label "CAN_Rx"
 		(at 229.87 113.03 0)
-		(fields_autoplaced yes)
 		(effects
 			(font
@@
 	(label "RCC_OSC_OUT"
 		(at 40.64 62.23 270)
-		(fields_autoplaced yes)
 		(effects
 			(font
@@
 	(label "RCC_OSC32_OUT"
 		(at 81.28 58.42 270)
-		(fields_autoplaced yes)
 		(effects
 			(font
@@
 	(label "BOOT1"
 		(at 165.1 90.17 0)
-		(fields_autoplaced yes)
 		(effects
 			(font
@@
 	(label "RCC_OSC_IN"
 		(at 19.05 63.5 270)
-		(fields_autoplaced yes)
 		(effects
 			(font
@@
 	(label "CAN_Tx"
 		(at 213.36 87.63 180)
-		(fields_autoplaced yes)
 		(effects
 			(font
@@
 	(label "CAN_Rx"
 		(at 213.36 85.09 180)
-		(fields_autoplaced yes)
 		(effects
 			(font
@@
 	(label "BOOT0"
 		(at 166.37 62.23 0)
-		(fields_autoplaced yes)
 		(effects
 			(font
@@
 	(label "RCC_OSC_IN"
 		(at 160.02 67.31 0)
-		(fields_autoplaced yes)
 		(effects
 			(font
@@
 	(label "RST"
 		(at 125.73 133.35 180)
-		(fields_autoplaced yes)
 		(effects
 			(font
@@
 	(label "BOOT0"
 		(at 15.24 134.62 0)
-		(fields_autoplaced yes)
 		(effects
 			(font
@@
 	(label "RCC_OSC32_OUT"
 		(at 156.21 80.01 0)
-		(fields_autoplaced yes)
 		(effects
 			(font
@@
 	(label "RCC_OSC32_IN"
 		(at 59.69 60.96 270)
-		(fields_autoplaced yes)
 		(effects
 			(font
@@
 	(label "3.3DCV"
 		(at 187.96 40.64 270)
-		(fields_autoplaced yes)
 		(effects
 			(font
@@
 	(label "RCC_OSC_OUT"
 		(at 158.75 69.85 0)
-		(fields_autoplaced yes)
 		(effects
 			(font
@@
 	(label "RST"
 		(at 167.64 57.15 0)
-		(fields_autoplaced yes)
 		(effects
 			(font
@@
 	(label "RCC_OSC32_IN"
 		(at 157.48 77.47 0)
-		(fields_autoplaced yes)
 		(effects
 			(font
@@
 		(shape input)
 		(at 33.02 27.94 180)
-		(fields_autoplaced yes)
+		(effects
+			(font
+				(size 1.27 1.27)
+			)
+			(justify right)
+		)
+	)
+	(hierarchical_label "ALERT_B_U"
+		(shape input)
+		(at 161.29 87.63 180)
+		(effects
+			(font
+				(size 1.27 1.27)
+			)
+			(justify right)
+		)
+	)
+	(hierarchical_label "CHG_DET"
+		(shape input)
+		(at 167.64 115.57 180)
 		(effects
 			(font
@@
 		(shape input)
 		(at 119.38 118.11 90)
-		(fields_autoplaced yes)
 		(effects
 			(font
@@
 		(shape input)
 		(at 170.18 100.33 180)
-		(fields_autoplaced yes)
 		(effects
 			(font
@@
 		(shape input)
 		(at 36.83 44.45 270)
-		(fields_autoplaced yes)
+		(effects
+			(font
+				(size 1.27 1.27)
+			)
+			(justify right)
+		)
+	)
+	(hierarchical_label "I2C_CTRL_U"
+		(shape input)
+		(at 158.75 92.71 180)
 		(effects
 			(font
@@
 		(shape input)
 		(at 246.38 102.87 180)
-		(fields_autoplaced yes)
 		(effects
 			(font
@@
 		(shape input)
 		(at 189.23 133.35 270)
-		(fields_autoplaced yes)
-		(effects
-			(font
-				(size 1.27 1.27)
-			)
-			(justify right)
+		(effects
+			(font
+				(size 1.27 1.27)
+			)
+			(justify right)
+		)
+	)
+	(hierarchical_label "I2C_CTRL_B_U"
+		(shape input)
+		(at 158.75 97.79 180)
+		(effects
+			(font
+				(size 1.27 1.27)
+			)
+			(justify right)
+		)
+	)
+	(hierarchical_label "I2C_CTRL_B"
+		(shape input)
+		(at 158.75 95.25 180)
+		(effects
+			(font
+				(size 1.27 1.27)
+			)
+			(justify right)
+		)
+	)
+	(hierarchical_label "LOAD_RM_DETECT"
+		(shape input)
+		(at 209.55 77.47 0)
+		(effects
+			(font
+				(size 1.27 1.27)
+			)
+			(justify left)
 		)
 	)
@@
 		(shape input)
 		(at 43.18 120.65 180)
-		(fields_autoplaced yes)
 		(effects
 			(font
@@
 		(shape input)
 		(at 130.81 81.28 270)
-		(fields_autoplaced yes)
 		(effects
 			(font
@@
 		(shape input)
 		(at 49.53 147.32 270)
-		(fields_autoplaced yes)
 		(effects
 			(font
@@
 		(shape input)
 		(at 58.42 96.52 270)
-		(fields_autoplaced yes)
+		(effects
+			(font
+				(size 1.27 1.27)
+			)
+			(justify right)
+		)
+	)
+	(hierarchical_label "ALERT_B"
+		(shape input)
+		(at 162.56 85.09 180)
 		(effects
 			(font
@@
 		(shape input)
 		(at 170.18 102.87 180)
-		(fields_autoplaced yes)
 		(effects
 			(font
@@
 		(shape input)
 		(at 248.92 129.54 270)
-		(fields_autoplaced yes)
-		(effects
-			(font
-				(size 1.27 1.27)
-			)
-			(justify right)
+		(effects
+			(font
+				(size 1.27 1.27)
+			)
+			(justify right)
+		)
+	)
+	(hierarchical_label "PDSG"
+		(shape input)
+		(at 215.9 59.69 0)
+		(effects
+			(font
+				(size 1.27 1.27)
+			)
+			(justify left)
 		)
 	)
@@
 		(shape input)
 		(at 102.87 148.59 270)
-		(fields_autoplaced yes)
 		(effects
 			(font
@@
 		(shape input)
 		(at 17.78 95.25 270)
-		(fields_autoplaced yes)
-		(effects
-			(font
+		(effects
+			(font

Commit message: Demo commit
Parts:
- C26, C27, C28, C29, C34: LCSC (none) -> C513772
Changed lines of the file:
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@@
 			)
 		)
-		(property "Datasheet" "~"
+		(property "Datasheet" "https://www.lcsc.com/datasheet/lcsc_datasheet_2410121935_Samwha-Capacitor-CS1005X7R104K500NR_C513772.pdf"
 			(at 69.85 35.56 0)
 			(effects
@@
 		)
 		(property "Sim.Pins" ""
+			(at 69.85 35.56 0)
+			(effects
+				(font
+					(size 1.27 1.27)
+				)
+				(hide yes)
+			)
+		)
+		(property "LCSC" "C513772"
 			(at 69.85 35.56 0)
 			(effects
@@
 			)
 		)
-		(property "Datasheet" "~"
+		(property "Datasheet" "https://www.lcsc.com/datasheet/lcsc_datasheet_2410121935_Samwha-Capacitor-CS1005X7R104K500NR_C513772.pdf"
 			(at 119.38 138.43 0)
 			(effects
@@
 		)
 		(property "Sim.Pins" ""
+			(at 119.38 138.43 0)
+			(effects
+				(font
+					(size 1.27 1.27)
+				)
+				(hide yes)
+			)
+		)
+		(property "LCSC" "C513772"
 			(at 119.38 138.43 0)
 			(effects
@@
 			)
 		)
-		(property "Datasheet" "~"
+		(property "Datasheet" "https://www.lcsc.com/datasheet/lcsc_datasheet_2410121935_Samwha-Capacitor-CS1005X7R104K500NR_C513772.pdf"
 			(at 59.69 35.56 0)
 			(effects
@@
 		)
 		(property "Sim.Pins" ""
+			(at 59.69 35.56 0)
+			(effects
+				(font
+					(size 1.27 1.27)
+				)
+				(hide yes)
+			)
+		)
+		(property "LCSC" "C513772"
 			(at 59.69 35.56 0)
 			(effects
@@
 			)
 		)
-		(property "Datasheet" "~"
+		(property "Datasheet" "https://www.lcsc.com/datasheet/lcsc_datasheet_2410121935_Samwha-Capacitor-CS1005X7R104K500NR_C513772.pdf"
 			(at 81.28 35.56 0)
 			(effects
@@
 		)
 		(property "Sim.Pins" ""
+			(at 81.28 35.56 0)
+			(effects
+				(font
+					(size 1.27 1.27)
+				)
+				(hide yes)
+			)
+		)
+		(property "LCSC" "C513772"
 			(at 81.28 35.56 0)
 			(effects
@@
 			)
 		)
-		(property "Datasheet" "~"
+		(property "Datasheet" "https://www.lcsc.com/datasheet/lcsc_datasheet_2410121935_Samwha-Capacitor-CS1005X7R104K500NR_C513772.pdf"
 			(at 48.26 35.56 0)
 			(effects
@@
 			(at 48.26 35.56 0)
 			(effects
+				(font
+					(size 1.27 1.27)
+				)
+				(hide yes)
+			)
+		)
+		(property "LCSC" "C513772"
+			(at 48.26 35.56 0)
+			(effects
