File: power.kicad_sch (KiCad schematic)
At the start: 22 parts, among them U6 AMS1117-3.3, U7 LM2596S-5

Commit message: Demo commit
Parts:
- C40, C42, C43, C45, C47, C48, C49: LCSC (none) -> C513772
Changed lines of the file:
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@@
+			)
+		)
+		(property "LCSC" "C513772"
+			(at 118.11 62.23 90)
+			(effects
+				(font
+					(size 1.27 1.27)
+				)
+				(hide yes)
 			)
 		)
@@
 			)
 		)
-		(property "Datasheet" "~"
+		(property "Datasheet" "https://www.lcsc.com/datasheet/lcsc_datasheet_2410121935_Samwha-Capacitor-CS1005X7R104K500NR_C513772.pdf"
 			(at 195.58 67.31 0)
 			(effects
@@
 		)
 		(property "Sim.Pins" ""
+			(at 195.58 67.31 0)
+			(effects
+				(font
+					(size 1.27 1.27)
+				)
+				(hide yes)
+			)
+		)
+		(property "LCSC" "C513772"
 			(at 195.58 67.31 0)
 			(effects
@@
 			)
 		)
-		(property "Datasheet" "~"
+		(property "Datasheet" "https://www.lcsc.com/datasheet/lcsc_datasheet_2410121935_Samwha-Capacitor-CS1005X7R104K500NR_C513772.pdf"
 			(at 102.87 96.52 0)
 			(effects
@@
 		(property "Sim.Pins" ""
 			(at 102.87 96.52 0)
+			(effects
+				(font
+					(size 1.27 1.27)
+				)
+				(hide yes)
+			)
+		)
+		(property "LCSC" "C513772"
+			(at 102.87 96.52 90)
 			(effects
 				(font
@@
 			)
 		)
+		(property "LCSC" "C513772"
+			(at 127 62.23 90)
+			(effects
+				(font
+					(size 1.27 1.27)
+				)
+				(hide yes)
+			)
+		)
 		(pin "2"
 		)
@@
 			)
 		)
-		(property "Datasheet" "~"
+		(property "Datasheet" "https://www.lcsc.com/datasheet/lcsc_datasheet_2410121935_Samwha-Capacitor-CS1005X7R104K500NR_C513772.pdf"
 			(at 209.55 68.58 0)
 			(effects
@@
 		)
 		(property "Sim.Pins" ""
+			(at 209.55 68.58 0)
+			(effects
+				(font
+					(size 1.27 1.27)
+				)
+				(hide yes)
+			)
+		)
+		(property "LCSC" "C513772"
 			(at 209.55 68.58 0)
 			(effects
@@
 			)
 		)
-		(property "Datasheet" "~"
+		(property "Datasheet" "https://www.lcsc.com/datasheet/lcsc_datasheet_2410121935_Samwha-Capacitor-CS1005X7R104K500NR_C513772.pdf"
 			(at 142.24 97.79 0)
 			(effects
@@
 		(property "Sim.Pins" ""
 			(at 142.24 97.79 0)
+			(effects
+				(font
+					(size 1.27 1.27)
+				)
+				(hide yes)
+			)
+		)
+		(property "LCSC" "C513772"
+			(at 142.24 97.79 90)
 			(effects
 				(font
@@
 			)
 		)
-		(property "Datasheet" "~"
+		(property "Datasheet" "https://www.lcsc.com/datasheet/lcsc_datasheet_2410121935_Samwha-Capacitor-CS1005X7R104K500NR_C513772.pdf"
 			(at 182.88 67.31 0)
 			(effects
@@
 			(at 182.88 67.31 0)
 			(effects
+				(font
+					(size 1.27 1.27)
+				)
+				(hide yes)
+			)
+		)
+		(property "LCSC" "C513772"
+			(at 182.88 67.31 0)
+			(effects
