File: Charge&discharge.kicad_sch (KiCad schematic)
At the start: 97 parts, among them Q1 NMOS, Q10 NMOS, Q11 NMOS, Q12 NMOS, Q13 NMOS, Q14 NMOS, Q15 NMOS, Q16 NMOS, Q17 NMOS, Q18 NMOS, Q19 NMOS, Q2 NMOS, Q20 NMOS, Q21 NMOS, Q22 NMOS, Q23 NMOS, Q24 NMOS, Q25 NMOS, Q26 NMOS, Q27 NMOS, Q28 NMOS, Q29 NMOS, Q3 NMOS, Q30 NMOS, Q31 NMOS, Q32 NMOS, Q33 NMOS, Q34 NMOS, Q35 NMOS, Q36 NMOS, Q37 NMOS, Q38 NMOS, Q39 NMOS, Q4 NMOS, Q40 NMOS, Q41 NMOS, Q5 NMOS, Q6 NMOS, Q7 NMOS, Q8 NMOS, Q9 NMOS

Commit message: second changes in bms monitoring
Connections:
- net GND is gone; now on net BAT-: D1.2 (A)
Changed lines of the file:
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@@
 	(wire
 		(pts
-			(xy 204.47 43.18) (xy 204.47 41.91)
+			(xy 204.47 41.91) (xy 204.47 44.45)
 		)
 		(stroke
@@
 		)
 	)
+	(hierarchical_label "BAT-"
+		(shape bidirectional)
+		(at 204.47 44.45 270)
+		(effects
+			(font
+				(size 1.27 1.27)
+			)
+			(justify right)
+		)
+	)
 	(hierarchical_label "PORT-"
 		(shape bidirectional)
@@
 					(unit 1)
 				)
-			)
-		)
-	)
-	(symbol
-		(lib_id "power:GND")
-		(at 204.47 43.18 0)
-		(unit 1)
-		(exclude_from_sim no)
-		(in_bom yes)
-		(on_board yes)
-		(dnp no)
-		(fields_autoplaced yes)
-		(property "Reference" "#PWR01"
-			(at 204.47 49.53 0)
-			(effects
-				(font
-					(size 1.27 1.27)
-				)
-				(hide yes)
-			)
-		)
-		(property "Value" "GND"
-			(at 204.47 48.26 0)
-			(effects
-				(font
-					(size 1.27 1.27)
-				)
-			)
-		)
-		(property "Footprint" ""
-			(at 204.47 43.18 0)
-			(effects
-				(font
-					(size 1.27 1.27)
-				)
-				(hide yes)
-			)
-		)
-		(property "Datasheet" ""
-			(at 204.47 43.18 0)
-			(effects
-				(font
-					(size 1.27 1.27)
-				)
-				(hide yes)
-			)
-		)
-		(property "Description" "Power symbol creates a global label with name \"GND\" , ground"
-			(at 204.47 43.18 0)
-			(effects
-				(font
-					(size 1.27 1.27)
-				)
-				(hide yes)
-			)
-		)
-		(pin "1"
-		)
-		(instances
-			(project ""
-				(path "/422fc8bd-c42e-475a-86fa-949c078f7358/5bba744b-5d77-4f20-8005-b356ef71a0a1"
-					(reference "#PWR01")
-					(unit 1)
-				)

Commit message: schematic v0
Parts:
- removed C1, C2, C3, C4: C, symbol Device:C
- removed D3, D4: D_Zener, symbol Device:D_Zener
- removed Q41: NMOS, symbol Simulation_SPICE:NMOS
- added C50, C51, C52: 0.1uF, symbol Device:C
- added Q41, Q62, Q63, Q64, Q65: NPN, symbol Simulation_SPICE:NPN
- added Q66: NMOS, symbol Simulation_SPICE:NMOS
- added R100, R101, R104, R105, R92, R93, R94, R95, R96, R97, R98, R99: 1k, symbol Device:R
- added R102, R103: 100, symbol Device:R
- added U10, U11, U8, U9: SFH617A-1, Package_DIP:DIP-4_W7.62mm, symbol Isolator:SFH617A-1
- C5, C6: value C -> 0.1uF
- R43: value 300u -> 0.001
Connections:
- net PORT+ is gone; now on net PORT-: C6.2, D6.2 (A), Q21.3 (S), Q22.3 (S), Q23.3 (S), Q24.3 (S), Q25.3 (S), Q26.3 (S), Q27.3 (S), Q28.3 (S), Q29.3 (S), Q30.3 (S), Q31.3 (S), Q32.3 (S), Q33.3 (S), Q34.3 (S), Q35.3 (S), Q36.3 (S), Q37.3 (S), Q38.3 (S), Q39.3 (S), Q40.3 (S), R60.2, R60.3
- net BAT-: now also R103.1
- net CHG+: now also D2.2 (A), Q66.3 (S); no longer D2.1 (K)
- net PDSG: now also R104.1; no longer D1.1 (K), R31.2
- net PORT-: no longer R43.2
- net at R60.1: now also Q66.1 (D)
- net at R31.1, R42.2: now also D2.1 (K), Q66.2 (G); no longer D2.2 (A)
- net BAT+: no longer names the net of C5.1, D5.2 (A), Q1.3 (S), Q10.3 (S), Q11.3 (S), Q12.3 (S), Q13.3 (S), Q14.3 (S), Q15.3 (S), Q16.3 (S), Q17.3 (S), Q18.3 (S), Q19.3 (S), Q2.3 (S), Q20.3 (S), Q3.3 (S), Q4.3 (S), Q5.3 (S), Q6.3 (S), Q7.3 (S), Q8.3 (S), Q9.3 (S)
- net BAT+: now also R43.2, R102.1
- net CHG renamed DSG_OR
- net DSG_OR: now also Q64.3 (E), Q65.3 (E), R101.2
- net DSG renamed CHG_OR
- net CHG_OR: now also Q62.3 (E), Q63.3 (E), R100.2
- new net: Q41.2 (B), R104.2
- new net: R94.2, U9.1
- new net: R92.2, U8.1
- new net: R96.2, U10.1
- new net: R97.2, U11.1
- new net CHG_B: R96.1
- new net CHG_B_B: Q63.2 (B), R98.2, U10.3
- new net CHG_U: R92.1
- new net CHG_U_B: Q62.2 (B), R93.2, U8.3
- new net DSG_B: R97.1
- new net DSG_B_B: Q65.2 (B), R99.2, U11.3
- new net DSG_U: R94.1
- new net DSG_U_B: Q64.2 (B), R95.2, U9.3
- new net GATE_TURN_ON: D1.1 (K), Q41.1 (C), R105.1, R31.2
- new net GND_B: C51.1, C52.2, Q41.3 (E), R100.1, R101.1, R93.1, R95.1, R98.1, R99.1, U10.2, U11.2
- new net GND_U: U8.2, U9.2
- new net Logic_ref: U10.4, U11.4, U8.4, U9.4
- new net SHUNT_N: C50.2, C52.1, R102.2
- new net SHUNT_P: C50.1, C51.2, R103.2
- new net Turn_ON _gate_V: Q62.1 (C), Q63.1 (C), Q64.1 (C), Q65.1 (C), R105.2
Other:
- note added: "LEVEL SHIFTER"
- note added: "OR-LOGIC"
- moved on the sheet: D1, D2, R31, R42, R60

Commit message: Demo commit
Parts:
- removed D2, D5, D6: D_Zener, symbol Device:D_Zener
- added D40: 1SMB5930B, easyeda2kicad:SMB_L4.8-W3.6-LS5.4-RD, symbol easyeda2kicad:1SMB5930B
- added U12, U13: BZT52C16_C2903915, easyeda2kicad:SOD-123_L2.7-W1.6-LS3.8-RD, symbol easyeda2kicad:BZT52C16_C2903915
- C5, C50, C51, C52, C6: footprint (none) -> Capacitor_SMD:C_0402_1005Metric; LCSC (none) -> C513772
Connections:
- net CHG+: now also D40.2
- net CHG_OR: now also U13.1 (K)
- net DSG_OR: now also U12.1 (K)
- net PORT-: now also U13.2 (A)
- net at C5.1, Q1.3 (S), Q10.3 (S)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: now also U12.2 (A)
- net at Q66.2 (G), R31.1, R42.2: now also D40.1

Commit message: MVP Friday
Parts:
- removed R60: 55, symbol Device:R_Potentiometer_Trim
- added R132: PWR163S-25-50R0J, PWR163S-25-50R0J:PWR163S2550R0F, symbol PWR136S-25-50R0J:PWR163S-25-50R0J
- R1, R10, R11, R12, R13, R14, R15, R16, R17, R18, R19, R2, R20, R21, R22, R23, R24, R25, R26, R27, R28, R29, R3, R30, R32, R33, R34, R35, R36, R37, R38, R39, R4, R40, R41, R5, R6, R7, R8, R9: footprint (none) -> Resistor_SMD:R_0201_0603Metric; LCSC (none) -> C7467289
- R31: footprint (none) -> Resistor_SMD:R_0805_2012Metric; LCSC (none) -> C407437
- R42: footprint (none) -> Resistor_SMD:R_0805_2012Metric; LCSC (none) -> C2771009
- R43: footprint (none) -> Resistor_SMD:R_2512_6332Metric; LCSC (none) -> C22383486
Connections:
- net PORT-: now also R132.2, R132.3
- net at Q66.1 (D): now also R132.1
