File: charger&load_detection.kicad_sch (KiCad schematic)
At the start: 31 parts, among them Q54 PMOS, Q55 NMOS, Q56 PMOS, Q57 NMOS, Q58 NMOS, Q59 PMOS

Commit message: Demo commit
Parts:
- removed 13V, 13V1: D_Zener, symbol Device:D_Zener
- added D3, D4: BZT52C12, easyeda2kicad:SOD-123_L2.7-W1.6-LS3.7-RD, symbol easyeda2kicad:BZT52C12
- C19: footprint (none) -> Capacitor_SMD:C_0603_1608Metric; LCSC (none) -> C513775
Connections:
- net at Q57.2 (G), R76.1: now also D4.1 (K)
- net at Q57.3 (S), R77.1: now also D4.2 (A)
- net at Q54.3 (S), Q55.3 (S), R74.1: now also D3.1 (K)
- net at Q54.2 (G), Q56.3 (S), R74.2: now also D3.2 (A)
Changed lines of the file:
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@@
-	)
-	(junction
-		(at 76.2 91.44)
-		(diameter 0)
-		(color 0 0 0 0)
 	)
 	(junction
@@
 	)
 	(junction
+		(at 77.47 91.44)
+		(diameter 0)
+		(color 0 0 0 0)
+	)
+	(junction
 		(at 72.39 59.69)
+		(diameter 0)
+		(color 0 0 0 0)
+	)
+	(junction
+		(at 67.31 102.87)
 		(diameter 0)
 		(color 0 0 0 0)
@@
 	)
 	(junction
-		(at 67.31 102.87)
-		(diameter 0)
-		(color 0 0 0 0)
-	)
-	(junction
 		(at 203.2 77.47)
 		(diameter 0)
@@
 	(wire
 		(pts
-			(xy 72.39 59.69) (xy 82.55 59.69)
+			(xy 72.39 59.69) (xy 86.36 59.69)
 		)
 		(stroke
@@
 	(wire
 		(pts
-			(xy 76.2 102.87) (xy 67.31 102.87)
+			(xy 67.31 102.87) (xy 77.47 102.87)
 		)
 		(stroke
@@
 	(wire
 		(pts
+			(xy 77.47 91.44) (xy 85.09 91.44)
+		)
+		(stroke
+			(width 0)
+			(type default)
+		)
+	)
+	(wire
+		(pts
 			(xy 63.5 97.79) (xy 63.5 101.6)
 		)
@@
 	(wire
 		(pts
-			(xy 82.55 60.96) (xy 82.55 59.69)
-		)
-		(stroke
-			(width 0)
-			(type default)
-		)
-	)
-	(wire
-		(pts
-			(xy 76.2 91.44) (xy 76.2 95.25)
+			(xy 82.55 69.85) (xy 86.36 69.85)
 		)
 		(stroke
@@
 	(wire
 		(pts
-			(xy 76.2 91.44) (xy 85.09 91.44)
+			(xy 74.93 91.44) (xy 77.47 91.44)
 		)
 		(stroke
@@
 	(wire
 		(pts
-			(xy 74.93 91.44) (xy 76.2 91.44)
-		)
-		(stroke
-			(width 0)
-			(type default)
-		)
-	)
-	(wire
-		(pts
 			(xy 165.1 67.31) (xy 170.18 67.31)
 		)
@@
 	(wire
 		(pts
-			(xy 82.55 68.58) (xy 82.55 69.85)
+			(xy 77.47 92.71) (xy 77.47 91.44)
 		)
 		(stroke
@@
 			)
 			(justify left)
+		)
+	)
+	(symbol
+		(lib_id "easyeda2kicad:BZT52C12")
+		(at 86.36 64.77 270)
+		(unit 1)
+		(exclude_from_sim no)
+		(in_bom yes)
+		(on_board yes)
+		(dnp no)
+		(fields_autoplaced yes)
+		(property "Reference" "D3"
+			(at 90.17 62.8649 90)
+			(effects
+				(font
+					(size 1.27 1.27)
+				)
+				(justify left)
+			)
+		)
+		(property "Value" "BZT52C12"
+			(at 90.17 65.4049 90)
+			(effects
+				(font
+					(size 1.27 1.27)
+				)
+				(justify left)
+			)
+		)
+		(property "Footprint" "easyeda2kicad:SOD-123_L2.7-W1.6-LS3.7-RD"
+			(at 78.74 64.77 0)
+			(effects
+				(font
+					(size 1.27 1.27)
+				)
+				(hide yes)
+			)
+		)
+		(property "Datasheet" "https://lcsc.com/product-detail/Zener-Diodes_BZT52C12_C173429.html"
+			(at 76.2 64.77 0)
+			(effects
+				(font
+					(size 1.27 1.27)
+				)
+				(hide yes)
+			)
+		)
+		(property "Description" ""
+			(at 86.36 64.77 0)
+			(effects
+				(font
+					(size 1.27 1.27)
+				)
+				(hide yes)
+			)
+		)
+		(property "LCSC Part" "C173429"
+			(at 73.66 64.77 0)
+			(effects
+				(font
+					(size 1.27 1.27)
+				)
+				(hide yes)
+			)
+		)
+		(pin "1"
+		)
+		(pin "2"
+		)
+		(instances
+			(project ""
+				(path "/422fc8bd-c42e-475a-86fa-949c078f7358/feaa7d91-301d-4a94-a100-c7358829192f"
+					(reference "D3")
+					(unit 1)
+				)
+			)
 		)
 	)
@@
 	)
 	(symbol
-		(lib_id "Device:D_Zener")
-		(at 76.2 99.06 270)
-		(unit 1)
-		(exclude_from_sim no)
-		(in_bom yes)
-		(on_board yes)
-		(dnp no)
-		(fields_autoplaced yes)
-		(property "Reference" "13V1"
-			(at 78.74 97.7899 90)
-			(effects
-				(font
-					(size 1.27 1.27)
-				)
-				(justify left)
-			)
-		)
-		(property "Value" "D_Zener"
-			(at 78.74 100.3299 90)
-			(effects
-				(font
-					(size 1.27 1.27)
-				)
-				(justify left)
-			)
-		)
-		(property "Footprint" ""
-			(at 76.2 99.06 0)
-			(effects
-				(font
-					(size 1.27 1.27)
-				)
-				(hide yes)
-			)
-		)
-		(property "Datasheet" "~"
-			(at 76.2 99.06 0)
-			(effects
-				(font
-					(size 1.27 1.27)
-				)
-				(hide yes)
-			)
-		)
-		(property "Description" "Zener diode"
-			(at 76.2 99.06 0)
-			(effects
-				(font
-					(size 1.27 1.27)
-				)
-				(hide yes)
-			)
-		)
-		(pin "1"
-		)
-		(pin "2"
-		)
-		(instances
-			(project "CustomBMS"
-				(path "/422fc8bd-c42e-475a-86fa-949c078f7358/feaa7d91-301d-4a94-a100-c7358829192f"
-					(reference "13V1")
-					(unit 1)
-				)
-			)
-		)
-	)
-	(symbol
 		(lib_id "Diode:1N4148W")
 		(at 33.02 102.87 270)
@@
 			)
 		)
-		(property "Footprint" ""
+		(property "Footprint" "Capacitor_SMD:C_0603_1608Metric"
 			(at 48.26 84.1248 0)
 			(effects
@@
 		(property "Description" "Unpolarized capacitor"
 			(at 44.45 85.09 0)
+			(effects
+				(font
+					(size 1.27 1.27)
+				)
+				(hide yes)
+			)
+		)
+		(property "LCSC" "C513775"
+			(at 44.45 85.09 90)
 			(effects
 				(font
@@
 				(path "/422fc8bd-c42e-475a-86fa-949c078f7358/feaa7d91-301d-4a94-a100-c7358829192f"
 					(reference "C19")
-					(unit 1)
-				)
-			)
-		)
-	)
-	(symbol
-		(lib_id "Device:D_Zener")
-		(at 82.55 64.77 270)
-		(unit 1)
-		(exclude_from_sim no)
-		(in_bom yes)
-		(on_board yes)
-		(dnp no)
-		(fields_autoplaced yes)
-		(property "Reference" "13V"
-			(at 85.09 63.4999 90)
-			(effects
-				(font
-					(size 1.27 1.27)
-				)
-				(justify left)
-			)
-		)
-		(property "Value" "D_Zener"
-			(at 85.09 66.0399 90)
-			(effects
-				(font
-					(size 1.27 1.27)
-				)
-				(justify left)
-			)
-		)
-		(property "Footprint" ""
-			(at 82.55 64.77 0)
-			(effects
-				(font
-					(size 1.27 1.27)
-				)
-				(hide yes)
-			)
-		)
-		(property "Datasheet" "~"
-			(at 82.55 64.77 0)
-			(effects
-				(font
-					(size 1.27 1.27)
-				)
-				(hide yes)
-			)
-		)
-		(property "Description" "Zener diode"
-			(at 82.55 64.77 0)
-			(effects
-				(font
-					(size 1.27 1.27)
-				)
-				(hide yes)
-			)
-		)
-		(pin "1"
-		)
-		(pin "2"
-		)
-		(instances
-			(project ""
-				(path "/422fc8bd-c42e-475a-86fa-949c078f7358/feaa7d91-301d-4a94-a100-c7358829192f"
-					(reference "13V")
 					(unit 1)
 				)
@@
 					(unit 1)
 				)
+			)
+		)
+	)
+	(symbol
+		(lib_id "easyeda2kicad:BZT52C12")
+		(at 77.47 97.79 270)
+		(unit 1)
+		(exclude_from_sim no)
+		(in_bom yes)
+		(on_board yes)
+		(dnp no)
+		(fields_autoplaced yes)
+		(property "Reference" "D4"
+			(at 81.28 95.8849 90)
+			(effects
+				(font
+					(size 1.27 1.27)
+				)
+				(justify left)
+			)
+		)
+		(property "Value" "BZT52C12"
+			(at 81.28 98.4249 90)
+			(effects
+				(font
+					(size 1.27 1.27)
+				)
+				(justify left)
+			)
+		)
+		(property "Footprint" "easyeda2kicad:SOD-123_L2.7-W1.6-LS3.7-RD"
+			(at 69.85 97.79 0)
+			(effects
+				(font
+					(size 1.27 1.27)
+				)
+				(hide yes)
+			)
+		)
+		(property "Datasheet" "https://lcsc.com/product-detail/Zener-Diodes_BZT52C12_C173429.html"
+			(at 67.31 97.79 0)
+			(effects
+				(font
+					(size 1.27 1.27)
+				)
+				(hide yes)
+			)
+		)
+		(property "Description" ""
+			(at 77.47 97.79 0)
+			(effects
+				(font
+					(size 1.27 1.27)
+				)
+				(hide yes)
+			)
+		)
+		(property "LCSC Part" "C173429"
+			(at 64.77 97.79 0)
+			(effects
+				(font
+					(size 1.27 1.27)
+				)
+				(hide yes)
+			)
+		)
+		(pin "1"
+		)
+		(pin "2"
+		)
+		(instances
+			(project "CustomBMS"
+				(path "/422fc8bd-c42e-475a-86fa-949c078f7358/feaa7d91-301d-4a94-a100-c7358829192f"
+					(reference "D4")
+					(unit 1)
+				)

Commit message: MVP Friday
Parts:
- removed D33, D34, D35: D_Zener, symbol Device:D_Zener
- added Z1, Z2, Z3: MMSZ5232BS-7-F, MMSZ5232BS-7-F:SOD2513X120N, symbol MMSZ5232BS-7-f:MMSZ5232BS-7-F
- R74: footprint (none) -> Resistor_SMD:R_0603_1608Metric; LCSC (none) -> C2907178
Connections:
- net BAT-: now also Z3.2 (A)
- net at D32.2 (A), R79.2: now also Z1.1 (K)
- new net: Z2.2 (A), Z3.1 (K)
- new net: Z1.2 (A), Z2.1 (K)
