File: monitoring.kicad_sch (KiCad schematic)
At the start: 65 parts, among them IC1 STM32F401RET6, Q42 NMOS, Q43 NMOS, Q44 PMOS, Q45 PMOS, Q46 PMOS, Q47 NMOS, Q48 NMOS, Q49 PMOS, Q50 NMOS, SW1 SW_Push, U1 BQ76940DBT, U2 BQ76940DBT, U3 ISO1541

Commit message: first change in bms monitoring
Parts:
- removed D17: 1N4148W, Diode_SMD:D_SOD-123, symbol Diode:1N4148W
- removed TH5: Thermistor, symbol Device:Thermistor
- added C20, C21: 4.7uF, symbol Device:C
- added C22: 4700pF, symbol Device:C
- added D17, D22: 13V, symbol Device:D_Zener
- added D20: 91V, symbol Device:D_Zener
- added D23: 1N4148W, Diode_SMD:D_SOD-123, symbol Diode:1N4148W
- added Q51, Q53: NMOS, symbol Simulation_SPICE:NMOS
- added Q52: PMOS, symbol Simulation_SPICE:PMOS
- added R65: 680k, symbol Device:R
- added R66: 1k, symbol Device:R
- added R67, R68, R70: 5.1M, symbol Device:R
- added R71: 1.2M, symbol Device:R
- added R72: 3M, symbol Device:R
- added TH7: Thermistor, symbol Device:Thermistor
- C17: value 4700pF -> 470pF
- R61: value 3M -> 510k
Connections:
- net SDA_B is gone; now on net SCL_B: Q42.1 (D), R57.2, U2.4 (SDA), U3.2 (SDA1)
- net GND_B: now also C20.2, D22.2 (A), R70.1, R71.2
- net GND_U: now also C17.2, R61.2, C21.2, R65.1
- net REGOUT_B: no longer U2.8 (REGOUT)
- net REGOUT_U: no longer U1.8 (REGOUT)
- net VC10_U: now also D16.2 (A)
- net VC5_U: now also D23.2 (A); no longer D16.2 (A)
- net VCC_B: now also U2.8 (REGOUT), C20.1, Q53.1 (D)
- net VCC_U: now also U1.8 (REGOUT), C21.1
- net at D14.2 (A), U1.24 (VC15): now also R66.2
- net TS3_U: now reaches C16.1, R59.1, TH2.1
- net TS3_U: now also U1.18 (TS3); no longer U1.13 (TS2)
- net VC10X_U: now reaches C16.2, D16.1 (K), R59.2, TH2.2
- net VC10X_U: now also U1.15 (VC10X); no longer U1.10 (VC5X)
- net Alert_B_U: now reaches IC1.56 (PB4)
- net Alert_B_U: now also Q53.3 (S), R71.1
- net Alertsignal_U: now reaches C17.1, R61.1
- net Alertsignal_U: now also U1.44 (ALERT), Q51.2 (G); no longer TH3.1, U1.18 (TS3)
- net TS2_B: now reaches C11.1, R52.1, U2.13 (TS2)
- net TS2_B: now also TH3.1
- net VC5X_B: now reaches C11.2, D12.1 (K), R52.2, U2.10 (VC5X)
- net VC5X_B: now also TH3.2
- net TS3_B: now reaches C12.1, R53.1, TH1.1, U2.18 (TS3)
- net VC10X_B: now reaches C12.2, D15.1 (K), R53.2, TH1.2, U2.15 (VC10X)
- net BATT+ renamed BAT+
- net BAT+: now also D17.1 (K), R66.1, R67.1, R68.1
- new net: D20.1 (K), Q52.3 (S), R68.2
- new net: Q51.1 (D), R67.2
- new net: Q51.3 (S), R65.2
- new net: D17.2 (A), Q52.2 (G)
- new net Alert_U: D20.2 (A), D22.1 (K), Q52.1 (D), Q53.2 (G), R70.2
- new net TS2_U: C22.1, R72.1, TH7.1, U1.13 (TS2)
- new net VC5X_U: C22.2, D23.1 (K), R72.2, TH7.2, U1.10 (VC5X)
Other:
- note added: "Alert connection- Upper"
- note added: "BMS IC Lower"
- note added: "BMS IC Upper"
- note added: "Isolator and logic change for I2C"
- note added: "Thermistor Connections- Lower"
- note added: "Thermistor Connections-Upper"
- moved on the sheet: C10, C13, C14, C15, C18, C7, C8, C9, D10, D11, D13, D14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

Commit message: second changes in bms monitoring
Parts:
- removed IC1: STM32F401RET6, QFP50P1200X1200X160-64N, symbol STM32f401REt6:STM32F401RET6
- removed Q43: NMOS, symbol Simulation_SPICE:NMOS
- removed Q44: PMOS, symbol Simulation_SPICE:PMOS
- added C23, C24: 1uF, symbol Device:C
- added D36, D37: 1N4148W, Diode_SMD:D_SOD-123, symbol Diode:1N4148W
- added Q43: PMOS, symbol Simulation_SPICE:PMOS
- added Q44, Q60, Q61: NMOS, symbol Simulation_SPICE:NMOS
- added R81, R82, R85: 200, symbol Device:R
- added R83, R84: 100, symbol Device:R
Connections:
- net BAT+: now also R81.1
- net GND_B: now also C24.1
- net GND_U: now also C23.1
- net I2C_CTRL_B: now also Q43.2 (G)
- net SCL_B: now also Q44.1 (D)
- net VC5X_B: now also R85.1
- net VC5X_U: now also R82.1
- net at C7.1, Q42.2 (G): now also Q43.1 (D), Q44.2 (G)
- net DSG_U: now reaches U1.1 (DSG)
- net CHG_U: now reaches U1.2 (CHG)
- net at U1.9 (REGSRC): now also C23.2, R83.2
- net Cell15: now reaches D13.2 (A), U2.24 (VC15)
- net Cell15: now also Q61.1 (D)
- net DSG_B: now reaches U2.1 (DSG)
- net CHG_B: now reaches U2.2 (CHG)
- net at U2.9 (REGSRC): now also C24.2, R84.2
- net VCC_B renamed SCL_MCU
- net SCL_MCU: now also Q43.3 (S), Q44.3 (S)
- new net: D37.1 (K), R84.1
- new net: D37.2 (A), Q61.3 (S)
- new net: Q61.2 (G), R85.2
- new net: Q60.1 (D), R81.2
- new net: Q60.2 (G), R82.2
- new net: D36.2 (A), Q60.3 (S)
- new net: D36.1 (K), R83.1
Other:
- note added: "I2C CONNECTION WITH MCU"
- moved on the sheet: C13, C14, C15, C17, C20, C21, D13, D14, D17, D20, D22, Q51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

Commit message: home changes
Parts:
- added R86, R87: 4.7k, symbol Device:R
Connections:
- net SCL_MCU: now also R87.2; no longer C20.1, D7.2 (A2), D9.2 (A2), Q42.3 (S), Q43.3 (S), Q45.3 (S), Q53.1 (D), U2.8 (REGOUT)
- new net SDA_MCU: Q42.3 (S), R86.2
- new net VCC_B: C20.1, D7.2 (A2), D9.2 (A2), Q43.3 (S), Q45.3 (S), Q53.1 (D), R86.1, R87.1, U2.8 (REGOUT)

Commit message: schematic v0
Parts:
- added C1, C2, C3, C4, C53, C54, C55, C56, C57, C58, C59, C60, C61, C62, C63, C64, C65, C66, C67, C68, C69, C70, C71, C72, C73, C74, C75: 220nF, symbol Device:C
- added R106, R107, R108, R109, R110, R111, R112, R113, R114, R115, R116, R117, R118, R119, R120, R121, R122, R123, R124, R125, R126, R127, R128, R129, R130, R131: 20, symbol Device:R
- R66: value 1k -> 20
Connections:
- net BAT+: now also D14.2 (A), U1.24 (VC15), C73.1
- net VC10X_B: now also C58.1, C59.2
- net VC10X_U: now also C70.1, C71.2
- net VC5X_B: now also C1.1, C54.2
- net VC5X_U: now also C66.2, C67.1
- net CELL_20: now reaches U1.25 (VC14)
- net CELL_20: now also U1.26 (VC13), U1.27 (VC12), C72.1, C73.2, R131.1
- net CELL_19: now reaches U1.28 (VC11)
- net CELL_19: now also C71.1, C72.2, R130.1
- net CELL_19_NEG: now reaches U1.29 (VC10B)
- net CELL_19_NEG: now also C70.2, R129.1
- net CELL_17: now reaches U1.31 (VC9)
- net CELL_17: now also U1.32 (VC8), U1.33 (VC7), C68.1, C69.2, R127.1
- net CELL_16: now reaches U1.34 (VC6)
- net CELL_16: now also C66.1, C68.2, R126.1
- net CELL_16_NEG: now reaches U1.35 (VC5B)
- net CELL_16_NEG: now also C67.2, R125.1
- net CELL_14: now reaches U1.37 (VC4)
- net CELL_14: now also U1.38 (VC3), C64.1, C65.2, R123.1
- net CELL_13: now reaches U1.39 (VC2)
- net CELL_13: now also C63.1, C64.2, R122.1
- net CELL_12_NEG: now reaches U1.41 (VC0)
- net CELL_12_NEG: now also C75.2, R120.1
- net CELL_10: now reaches U2.25 (VC14)
- net CELL_10: now also U2.26 (VC13), U2.27 (VC12), C60.1, C61.2, R118.1
- net CELL_9: now reaches U2.28 (VC11)
- net CELL_9: now also C59.1, C60.2, R117.1
- net CELL_9_NEG: now reaches U2.29 (VC10B)
- net CELL_9_NEG: now also C58.2, R116.1
- net CELL_7: now reaches U2.31 (VC9)
- net CELL_7: now also U2.32 (VC8), C56.1, C57.2, R114.1
- net CELL_6: now reaches U2.33 (VC7)
- net CELL_6: now also C55.1, C56.2, R113.1
- net CELL_5: now reaches U2.34 (VC6)
- net CELL_5: now also C54.1, C55.2, R106.1
- net CELL_5_NEG: now reaches U2.35 (VC5B)
- net CELL_5_NEG: now also C1.2, R112.1
- net CELL_3: now reaches U2.37 (VC4)
- net CELL_3: now also U2.38 (VC3), C2.2, C3.1, R109.1
- net CELL_2: now reaches U2.39 (VC2)
- net CELL_2: now also C3.2, C4.1, R110.1
- net CELL_1_NEG: now reaches U2.41 (VC0)
- net CELL_1_NEG: now also C74.2, R111.1
- net Cell15 renamed CELL_11
- net CELL_11: now also C61.1, R119.1
- net I_N renamed SHUNT_N
- net I_P renamed SHUNT_P
- net VC10_B renamed CELL_8
- net CELL_8: now also C57.1, R115.1
- net VC10_U renamed CELL_18
- net CELL_18: now also C69.1, R128.1
- net VC1_B renamed CELL_1
- net CELL_1: now also C4.2, C53.1, R108.1
- net VC1_U renamed CELL_12
- net CELL_12: now also C62.1, C63.2, R121.1
- net VC5_B renamed CELL_4
- net CELL_4: now also C2.1, R107.1
- net VC5_U renamed CELL_15
- net CELL_15: now also C65.1, R124.1
- new net: C62.2, C75.1
- new net: C53.2, C74.1
- new net BATT_1+: R108.2
- new net BATT_10+: R118.2
- new net BATT_11+: R119.2, R120.2
- new net BATT_12+: R121.2
- new net BATT_13+: R122.2
- new net BATT_14+: R123.2
- new net BATT_15+: R124.2, R125.2
- new net BATT_16+: R126.2
- new net BATT_17+: R127.2
- new net BATT_18+: R128.2, R129.2
- new net BATT_19+: R130.2
- new net BATT_1_NEG: R111.2
- new net BATT_2+: R110.2
- new net BATT_20+: R131.2
- new net BATT_21+: R66.2
- new net BATT_3+: R109.2
- new net BATT_4+: R107.2, R112.2
- new net BATT_5+: R106.2
- new net BATT_6+: R113.2
- new net BATT_7+: R114.2
- new net BATT_8+: R115.2, R116.2
- new net BATT_9+: R117.2
Other:
- moved on the sheet: C21

Commit message: Demo commit
Parts:
- removed D17: 13V, symbol Device:D_Zener
- removed D19: D_Zener, symbol Device:D_Zener
- added D17, D2: 13V, easyeda2kicad:SOD-123_L2.7-W1.6-LS3.7-RD, symbol easyeda2kicad:BZT52C12
- C1, C2, C3, C4, C53, C54, C55, C56, C57, C58, C59, C60, C61, C62, C63, C64, C65, C66, C67, C68, C69, C70, C71, C72, C73, C74, C75: footprint (none) -> Capacitor_SMD:C_0402_1005Metric; LCSC (none) -> C7503518
- C10, C11, C12, C16, C18, C22: footprint (none) -> Capacitor_SMD:C_0402_1005Metric; LCSC (none) -> C7503510
- C13, C15, C23, C24: footprint (none) -> Capacitor_SMD:C_0603_1608Metric; LCSC (none) -> C513775
- C14, C17: footprint (none) -> Capacitor_SMD:C_0201_0603Metric
- C7, C9: footprint (none) -> Capacitor_SMD:C_0402_1005Metric; LCSC (none) -> C513772
- C8: footprint (none) -> Capacitor_SMD:C_0402_1005Metric; LCSC part no (none) -> C513772
Connections:
- net GND_B is gone; now on net BATT_1_NEG: C10.1, C13.2, C14.2, C20.2, C24.1, C7.2, C8.2, D22.2 (A), R47.2, R49.1, R50.1, R51.1, R54.2, R70.1, R71.2, TH4.1, U2.3 (VSS), U3.4 (GND1)
- net GND_U is gone; now on net BATT_11+: C15.2, C17.2, C18.2, C21.2, C23.1, C9.2, D10.2 (A), R46.2, R61.2, R62.2, R65.1, TH6.2, U1.3 (VSS), U1.42 (SRP), U1.43 (SRN), U3.5 (GND2)
- net BAT+: now also D2.1 (K)
- net BATT_11+: now also C62.2, C75.1
- net BATT_1_NEG: now also C53.2, C74.1
- net TS1_U_CTRL: now also D17.2 (A)
- net at Q49.3 (S), Q50.1 (D), R64.2: now also D17.1 (K)
- net at Q52.2 (G): now also D2.2 (A)

Commit message: MVP Friday
Parts:
- C20, C21: footprint (none) -> Capacitor_SMD:C_1206_3216Metric; LCSC (none) -> C5189849
- R44, R45, R55, R56, R57, R58, R86, R87: footprint (none) -> Resistor_SMD:R_0603_1608Metric; LCSC (none) -> C2077906
- R46: footprint (none) -> Resistor_SMD:R_0603_1608Metric; LCSC (none) -> C103548
- R47: footprint (none) -> Resistor_SMD:R_0603_1608Metric; LCSC (none) -> C2930043
- R48, R50: footprint (none) -> Resistor_SMD:R_0402_1005Metric; LCSC (none) -> C325551
- R49, R51, R52, R53, R59, R62, R72: footprint (none) -> Resistor_SMD:R_0603_1608Metric; LCSC (none) -> C23156
- R54, R61: footprint (none) -> Resistor_SMD:R_0603_1608Metric; LCSC (none) -> C2907178
